File: hardware/logicboard/bma-001.brd (EAGLE design)
At the start: 47 x 72 mm, 3 parts

Commit message: First working model.
Parts:
- added J0: (no value), con-jack:SPC4077
- added J7, J8, J9: DIN5, SparkFun-Connectors:DIN5-RA-PTH
- added X0: MKDSN1,5/2-5,08, con-phoenix-508:MKDSN1,5/2-5,08
Connections:
- net GND: now also J0.1, J0.2, J8.2, J9.2, X0.1
- net MIRTN: now also J7.5
- net MISND: now also J7.4
- net MORTN: now also J9.5
- net MOSND: now also J9.4
- net MTRTN: now also J8.5
- net MTSND: now also J8.4
- net V+: now also J0.3, X0.2
Routing:
- net GND: track 0.00 -> 110.1 mm
- net V+: track 0.00 -> 49.6 mm
- net MOSND: track 0.00 -> 36.5 mm
- net MIRTN: track 0.00 -> 34.0 mm
- net MTRTN: track 0.00 -> 28.0 mm
- net MISND: track 0.00 -> 25.2 mm
- net MTSND: track 0.00 -> 22.8 mm
- net MORTN: track 0.00 -> 22.1 mm
- added copper zone on layer 1, net GND
- added copper zone on layer 16, net GND
Other:
- board text added: "+"
- board text added: "-"
- board text added: "Backport MIDI Adapter 0.0.1-X"
- board text added: "DC12V"
- board text added: "MIDI IN"
- board text added: "MIDI OUT"
- board text added: "MIDI THRU"
