File: hardware/logicboard/bma-001.sch (EAGLE design)
At the start: 3 parts

Commit message: First working model.
Parts:
- added J0: (no value), con-jack:JACK-PLUG0
- added J7, J8, J9: DIN5, SparkFun-Connectors:DIN5
- added X0: MKDSN1,5/2-5,08, con-phoenix-508:MKDSN1,5/2-5,08
Connections:
- net GND: now also J0.1, J0.2, J8.2, J9.2, X0-1.KL
- net MIRTN: now also J7.5
- net MISND: now also J7.4
- net MORTN: now also J9.5
- net MOSND: now also J9.4
- net MTRTN: now also J8.5
- net MTSND: now also J8.4
- net V+: now also J0.3, X0-2.KL
Changed lines of the file:
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@@
 <part name="FRAME2" library="frames" library_urn="urn:adsk.eagle:library:229" deviceset="A3L-LOC" device=""/>
 <part name="SV2" library="con-ml" library_urn="urn:adsk.eagle:library:164" deviceset="ML20LE" device="" package3d_urn="urn:adsk.eagle:package:8685/1"/>
+<part name="J7" library="SparkFun-Connectors" library_urn="urn:adsk.eagle:library:513" deviceset="DIN5" device="" package3d_urn="urn:adsk.eagle:package:38294/1"/>
+<part name="J9" library="SparkFun-Connectors" library_urn="urn:adsk.eagle:library:513" deviceset="DIN5" device="" package3d_urn="urn:adsk.eagle:package:38294/1"/>
+<part name="J8" library="SparkFun-Connectors" library_urn="urn:adsk.eagle:library:513" deviceset="DIN5" device="" package3d_urn="urn:adsk.eagle:package:38294/1"/>
+<part name="J0" library="con-jack" library_urn="urn:adsk.eagle:library:154" deviceset="JACK-PLUG" device="0" package3d_urn="urn:adsk.eagle:package:7492/1"/>
+<part name="X0" library="con-phoenix-508" library_urn="urn:adsk.eagle:library:176" deviceset="MKDSN1,5/2-5,08" device="" package3d_urn="urn:adsk.eagle:package:9630/1"/>
 </parts>
 <sheets>
@@
 <attribute name="VALUE" x="319.786" y="85.979" size="1.778" layer="96"/>
 </instance>
+<instance part="J7" gate="G$1" x="266.7" y="160.02" smashed="yes">
+<attribute name="NAME" x="266.7" y="154.432" size="1.778" layer="95" font="vector" align="bottom-center"/>
+<attribute name="VALUE" x="266.7" y="152.146" size="1.778" layer="96" font="vector" align="top-center"/>
+</instance>
+<instance part="J9" gate="G$1" x="266.7" y="127" smashed="yes">
+<attribute name="NAME" x="266.7" y="121.412" size="1.778" layer="95" font="vector" align="bottom-center"/>
+<attribute name="VALUE" x="266.7" y="119.126" size="1.778" layer="96" font="vector" align="top-center"/>
+</instance>
+<instance part="J8" gate="G$1" x="269.24" y="91.44" smashed="yes">
+<attribute name="NAME" x="269.24" y="85.852" size="1.778" layer="95" font="vector" align="bottom-center"/>
+<attribute name="VALUE" x="269.24" y="83.566" size="1.778" layer="96" font="vector" align="top-center"/>
+</instance>
+<instance part="J0" gate="G$1" x="261.62" y="198.12" smashed="yes">
+<attribute name="NAME" x="254" y="203.2" size="1.778" layer="95"/>
+<attribute name="VALUE" x="254" y="193.04" size="1.778" layer="96"/>
+</instance>
+<instance part="X0" gate="-1" x="307.34" y="200.66" smashed="yes">
+<attribute name="NAME" x="310.388" y="199.771" size="1.778" layer="95"/>
+<attribute name="VALUE" x="304.8" y="196.977" size="1.778" layer="96"/>
+</instance>
+<instance part="X0" gate="-2" x="307.34" y="195.58" smashed="yes">
+<attribute name="NAME" x="310.388" y="194.691" size="1.778" layer="95"/>
+<attribute name="VALUE" x="304.8" y="191.897" size="1.778" layer="96"/>
+</instance>
 </instances>
 <busses>
@@
 <label x="314.96" y="142.24" size="0.8128" layer="95" rot="R180" xref="yes"/>
 </segment>
+<segment>
+<pinref part="J0" gate="G$1" pin="1"/>
+<wire x1="266.7" y1="195.58" x2="269.24" y2="195.58" width="0.1524" layer="91"/>
+<pinref part="J0" gate="G$1" pin="2"/>
+<wire x1="269.24" y1="195.58" x2="271.78" y2="195.58" width="0.1524" layer="91"/>
+<wire x1="266.7" y1="198.12" x2="269.24" y2="198.12" width="0.1524" layer="91"/>
+<wire x1="269.24" y1="198.12" x2="269.24" y2="195.58" width="0.1524" layer="91"/>
+<junction x="269.24" y="195.58"/>
+<label x="271.78" y="195.58" size="0.8128" layer="95" xref="yes"/>
+</segment>
+<segment>
+<pinref part="J9" gate="G$1" pin="2"/>
+<wire x1="266.7" y1="137.16" x2="266.7" y2="142.24" width="0.1524" layer="91"/>
+<label x="266.7" y="142.24" size="0.8128" layer="95" rot="R90" xref="yes"/>
+</segment>
+<segment>
+<pinref part="J8" gate="G$1" pin="2"/>
+<wire x1="269.24" y1="101.6" x2="269.24" y2="104.14" width="0.1524" layer="91"/>
+<label x="269.24" y="104.14" size="0.8128" layer="95" rot="R90" xref="yes"/>
+</segment>
+<segment>
+<pinref part="X0" gate="-1" pin="KL"/>
+<wire x1="304.8" y1="200.66" x2="302.26" y2="200.66" width="0.1524" layer="91"/>
+<label x="302.26" y="200.66" size="0.8128" layer="95" rot="R180" xref="yes"/>
+</segment>
 </net>
 <net name="VCC" class="2">
@@
 <label x="314.96" y="127" size="0.8128" layer="95" rot="MR0" xref="yes"/>
 </segment>
+<segment>
+<pinref part="J7" gate="G$1" pin="4"/>
+<wire x1="274.32" y1="165.1" x2="281.94" y2="165.1" width="0.1524" layer="91"/>
+<label x="281.94" y="165.1" size="0.8128" layer="95" xref="yes"/>
+</segment>
 </net>
 <net name="MIRTN" class="4">
@@
 <label x="314.96" y="119.38" size="0.8128" layer="95" rot="MR0" xref="yes"/>
 </segment>
+<segment>
+<pinref part="J7" gate="G$1" pin="5"/>
+<wire x1="259.08" y1="165.1" x2="251.46" y2="165.1" width="0.1524" layer="91"/>
+<label x="251.46" y="165.1" size="0.8128" layer="95" rot="R180" xref="yes"/>
+</segment>
 </net>
 <net name="MORTN" class="0">
@@
 <label x="314.96" y="99.06" size="0.8128" layer="95" rot="MR0" xref="yes"/>
 </segment>
+<segment>
+<pinref part="J9" gate="G$1" pin="5"/>
+<wire x1="259.08" y1="132.08" x2="254" y2="132.08" width="0.1524" layer="91"/>
+<label x="254" y="132.08" size="0.8128" layer="95" rot="R180" xref="yes"/>
+</segment>
 </net>
 <net name="MOSND" class="0">
@@
 <label x="314.96" y="111.76" size="0.8128" layer="95" rot="MR0" xref="yes"/>
 </segment>
+<segment>
+<pinref part="J9" gate="G$1" pin="4"/>
+<wire x1="274.32" y1="132.08" x2="279.4" y2="132.08" width="0.1524" layer="91"/>
+<label x="279.4" y="132.08" size="0.8128" layer="95" xref="yes"/>
+</segment>
 </net>
 <net name="V+" class="5">
@@
 <label x="314.96" y="154.94" size="0.8128" layer="95" rot="MR0" xref="yes"/>
 </segment>
+<segment>
+<pinref part="J0" gate="G$1" pin="3"/>
+<wire x1="266.7" y1="200.66" x2="271.78" y2="200.66" width="0.1524" layer="91"/>
+<label x="271.78" y="200.66" size="0.8128" layer="95" xref="yes"/>
+</segment>
+<segment>
+<pinref part="X0" gate="-2" pin="KL"/>
+<wire x1="304.8" y1="195.58" x2="302.26" y2="195.58" width="0.1524" layer="91"/>
+<label x="302.26" y="195.58" size="0.8128" layer="95" rot="R180" xref="yes"/>
+</segment>
 </net>
 <net name="MTSND" class="0">
@@
 <label x="314.96" y="109.22" size="0.8128" layer="95" rot="MR0" xref="yes"/>
 </segment>
+<segment>
+<pinref part="J8" gate="G$1" pin="4"/>
+<wire x1="276.86" y1="96.52" x2="281.94" y2="96.52" width="0.1524" layer="91"/>
+<label x="281.94" y="96.52" size="0.8128" layer="95" xref="yes"/>
+</segment>
 </net>
 <net name="MTRTN" class="0">
@@
 <label x="314.96" y="96.52" size="0.8128" layer="95" rot="MR0" xref="yes"/>
 </segment>
-</net>
+<segment>
+<pinref part="J8" gate="G$1" pin="5"/>
+<wire x1="261.62" y1="96.52" x2="254" y2="96.52" width="0.1524" layer="91"/>
+<label x="254" y="96.52" size="0.8128" layer="95" rot="R180" xref="yes"/>
+</segment>
+</net>
